File: macro-pad.sch (KiCad schematic (older format))
At the start: 14 parts

Commit message: added some footnotes
Parts:
- added D1, D2, D3, D4: SOD-123, Diode_SMD:D_SOD-123, symbol Device:D_Small
- added F1: 500mA, Fuse:Fuse_1206_3216Metric, symbol Device:Polyfuse_Small
- added MX1, MX2, MX3, MX4: MX-NoLED, MX_Only:MXOnly-1U-NoLED, symbol MX_Alps_Hybrid:MX-NoLED
- added USB1: Molex-0548190589, symbol random-keyboard-parts:Molex-0548190589
- C1, C2, C3, C4, C5, C6, C7: renamed from C?; footprint (none) -> Capacitor_SMD:C_0805_2012Metric
- R1, R2, R3, R4: renamed from R?; footprint (none) -> Resistor_SMD:R_0805_2012Metric
- Y1: renamed from Y?; footprint (none) -> Crystal:Crystal_SMD_3225-4Pin_3.2x2.5mm
- gave numbers to parts that had none: 2
Connections:
- net labels added: COL0, COL1, D+, D-, ROW0, ROW1, VCC
- wire segments 43 -> 59
